File: _autosave-sixtyfive.kicad_pcb (KiCad board)
At the start: 2 copper layers, 197 parts, among them J1 Conn_01x12, Q1 BSS138, U1 USBLC6-2SC6, U2 STM32F072C8Tx, U3 MCP1700-3302E_SOT23

Commit message: Placed all the switches, all the diodes!
Parts:
- added D67: D_Small, Diode_SMD:D_SOD-123, B.Cu at (142.9, 279.4)
- added D68: D_Small, Diode_SMD:D_SOD-123, B.Cu at (214.3, 279.4)
- added MX67: LSpace, MX_Only:MXOnly-2.75U-Hotswap-ReversedStabilizers, F.Cu at (147.6, 283.4)
- added MX68: RSpace, MX_Only:MXOnly-2.25U-Hotswap-ReversedStabilizers, F.Cu at (219.1, 283.4)
- added MX69: 125_Space, MX_Only:MXOnly-1.25U-Hotswap, F.Cu at (185.7, 283.4)
- CB1, D1, D10, D11, D12, D13, D14, D15, D16, D17, D18, D19, D2, D20, D21, D22, D23, D24, D25, D26, D27, D28, D29, D3, D30, D31, D32, D33, D34, D35, D36, D37, D38, D39, D4, D40, D41, D42, D43, D44, D45, D46, D47, D48, D49, D5, D50, D51, D52, D53, D54, D55, D56, D57, D58, D59, D6, D60, D61, D62, D63, D64, D65, D66, D7, D8, D9, J1, U2: moved to B.Cu
- moved RRGB3 633.5 mm to (521.9, 341.4)
- moved CB6 633.5 mm to (424.3, 338.6)
- moved CB7 633.5 mm to (424.3, 336.6)
- moved CB8 633.5 mm to (499.8, 257.2)
- moved CR1 633.5 mm to (369.4, 287.8)
- moved CR2 633.5 mm to (369.4, 281.9)
- moved CRGB2 633.5 mm to (369.2, 298.3)
- moved CRGB4 633.5 mm to (425.1, 331.2)
- moved CRGB5 633.5 mm to (425.1, 328.2)
- moved CRGB6 633.5 mm to (425.1, 325.3)
- moved CRGB7 633.5 mm to (425.1, 322.3)
- moved CSI1 633.5 mm to (369.4, 290.8)
- moved CSO1 633.5 mm to (369.4, 284.9)
- moved DRGB1 633.5 mm to (491.2, 269.6)
- moved DRGB3 633.5 mm to (491.2, 262.9)
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