File: sixtyfive.kicad_pcb (KiCad board)
At the start: 2 copper layers, 197 parts, among them J1 Conn_01x12, Q1 BSS138, U1 USBLC6-2SC6, U2 STM32F072C8Tx, U3 MCP1700-3302E_SOT23

Commit message: Placed rgb leds
Parts:
- added D67: D_Small, Diode_SMD:D_SOD-123, B.Cu at (142.9, 279.4)
- added D68: D_Small, Diode_SMD:D_SOD-123, B.Cu at (214.3, 279.4)
- added MX67: LSpace, MX_Only:MXOnly-2.75U-Hotswap-ReversedStabilizers, F.Cu at (147.6, 283.4)
- added MX68: RSpace, MX_Only:MXOnly-2.25U-Hotswap-ReversedStabilizers, F.Cu at (219.1, 283.4)
- added MX69: 125_Space, MX_Only:MXOnly-1.25U-Hotswap, F.Cu at (185.7, 283.4)
- CB1, CB2, CB3, CB4, CB5, CB6, CB7, CB8, CRGB1, CRGB10, CRGB2, CRGB3, CRGB4, CRGB5, CRGB6, CRGB7, CRGB8, CRGB9, D1, D10, D11, D12, D13, D14, D15, D16, D17, D18, D19, D2, D20, D21, D22, D23, D24, D25, D26, D27, D28, D29, D3, D30, D31, D32, D33, D34, D35, D36, D37, D38, D39, D4, D40, D41, D42, D43, D44, D45, D46, D47, D48, D49, D5, D50, D51, D52, D53, D54, D55, D56, D57, D58, D59, D6, D60, D61, D62, D63, D64, D65, D66, D7, D8, D9, DRGB1, DRGB10, DRGB2, DRGB3, DRGB4, DRGB5, DRGB6, DRGB7, DRGB8, DRGB9, J1, RRGB1, RRGB10, RRGB2, RRGB3, RRGB4, RRGB5, RRGB6, RRGB7, RRGB8, RRGB9, U1, U2: moved to B.Cu
- moved CR1 633.5 mm to (369.4, 287.8)
- moved CR2 633.5 mm to (369.4, 281.9)
- moved CSI1 633.5 mm to (369.4, 290.8)
- moved CSO1 633.5 mm to (369.4, 284.9)
- moved F1 633.5 mm to (490.4, 275.3)
- moved QRST1 633.5 mm to (369.2, 294.5)
- moved RSH1 633.5 mm to (531.4, 331.3)
- moved DS1 633.5 mm to (531.5, 328.0)
- moved U3 633.5 mm to (373.7, 295.1)
- moved CSH1 622.9 mm to (443.9, 248.9)
- moved CSH2 617.1 mm to (433.9, 249.4)
- moved Q1 600.8 mm to (418.8, 238.2)
- moved MX28 555.8 mm to (321.5, 226.2)
- moved MX64 552.4 mm to (326.2, 283.4)
- moved D56 543.4 mm to (350.0, 268.3), turned to 90 degrees
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
Commit message: Pretty sure I wired up the whole matrix
Parts:
- CSH1, CSH2, CSI1, CSO1, DF1, DS1, F1, Q1, RCC1, RCC2, RS1, RS2, RSH1, RSH2, RSO1, U3: moved to B.Cu
- moved DS1 469.1 mm to (76.4, 214.2), turned to 90 degrees
- moved F1 426.3 mm to (68.6, 213.6), turned to 90 degrees
- moved RSH1 424.7 mm to (128.2, 198.1), turned to 270 degrees
- moved CSH2 372.1 mm to (65.4, 197.0), turned to 270 degrees
- moved RCC2 358.3 mm to (58.9, 197.2), turned to 180 degrees
- moved RSH2 348.5 mm to (63.1, 197.6), turned to 90 degrees
- moved Q1 333.6 mm to (86.1, 213.2), turned to 180 degrees
- moved CSH1 322.5 mm to (125.4, 198.1), turned to 90 degrees
- moved RCC1 315.2 mm to (83.7, 197.4), turned to 180 degrees
- moved RSO1 314.1 mm to (83.2, 210.8), turned to 90 degrees
- moved RS2 309.1 mm to (78.0, 222.9), turned to 270 degrees
- moved U3 305.1 mm to (79.3, 214.9)
- moved CSI1 304.9 mm to (74.1, 214.8), turned to 90 degrees
- moved RS1 300.0 mm to (83.2, 215.8), turned to 270 degrees
- moved CSO1 297.7 mm to (80.9, 211.0), turned to 90 degrees
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Connections:
- J1 pad 12: Extra11 -> Extra12
- U2 pad 13: Row5 -> Col14
- U2 pad 14: Col14 -> Col13
- U2 pad 15: Col13 -> Col12
- U2 pad 16: LED_PWM -> Col11
- U2 pad 17: Col12 -> Col10
- U2 pad 19: Col10 -> Row5
- U2 pad 20: Col11 -> Row4
- U2 pad 22: Row4 -> Extra13
- U2 pad 28: RGB3V3 -> RGB_3V3
- U2 pad 3: Col7 -> Col8
- U2 pad 4: Col8 -> Col7
- U2 pad 5: Col5 -> Col6
- U2 pad 6: Col6 -> Col5
Routing:
- net Row1: track 0.00 -> 389.0 mm
- net Row5: track 0.00 -> 385.9 mm
- net Col14: track 0.00 -> 362.0 mm, vias 0 -> 4
- net Col13: track 0.00 -> 346.2 mm, vias 0 -> 2
- net Col12: track 0.00 -> 325.2 mm, vias 0 -> 6
- net Row3: track 0.00 -> 301.1 mm, vias 0 -> 26
- net Col10: track 0.00 -> 274.0 mm, vias 0 -> 2
- net Row2: track 0.00 -> 267.2 mm, vias 0 -> 25
- net Col11: track 0.00 -> 260.7 mm, vias 0 -> 2
- net Col9: track 0.00 -> 252.0 mm, vias 0 -> 4
- net Col7: track 0.00 -> 211.7 mm, vias 0 -> 2
- net Col8: track 0.00 -> 211.6 mm, vias 0 -> 4
- net Col4: track 0.00 -> 150.7 mm, vias 0 -> 2
- net Col6: track 0.00 -> 142.4 mm, vias 0 -> 4
- net Col5: track 0.00 -> 123.2 mm, vias 0 -> 2
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Other:
- net class Power added: clearance 0.2, trace_width 0.5, via_dia 0.8, via_drill 0.4

Commit message: Matrix rewired to allow for 5v line for rgb, which is also wired up
Parts:
- RSI1: moved to B.Cu
- moved RSI1 342.5 mm to (87.4, 207.7), turned to 90 degrees
- moved RRGB6 230.0 mm to (319.4, 271.2), turned to 90 degrees
- moved DRGB10 226.6 mm to (89.8, 271.1), turned to 180 degrees
- moved CRGB6 225.5 mm to (317.1, 270.5), turned to 90 degrees
- moved CRGB10 217.2 mm to (94.5, 270.4), turned to 90 degrees
- moved DRGB6 216.1 mm to (312.4, 271.2), turned to 180 degrees
- moved RRGB10 212.6 mm to (96.7, 270.9), turned to 90 degrees
- moved DRGB9 137.0 mm to (133.0, 271.2), turned to 180 degrees
- moved CRGB9 127.6 mm to (137.7, 270.5), turned to 90 degrees
- moved RRGB9 123.1 mm to (140.0, 271.2), turned to 90 degrees
- moved RRGB7 105.3 mm to (254.2, 271.1), turned to 90 degrees
- moved CRGB7 100.7 mm to (251.9, 270.5), turned to 90 degrees
- moved DRGB7 91.3 mm to (247.2, 271.1), turned to 180 degrees
- moved DRGB8 23.1 mm to (190.9, 271.1), turned to 180 degrees
- moved CRGB8 13.8 mm to (195.6, 270.4), turned to 90 degrees
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Routing:
- net 5V: track 15.1 -> 606.0 mm
- net Row4: track 82.9 -> 319.8 mm, vias 4 -> 16
- net Net-(DRGB5-Pad2): track 0.00 -> 103.8 mm, vias 0 -> 2
- net Net-(DRGB6-Pad2): track 0.00 -> 72.1 mm
- net Net-(DRGB8-Pad2): track 0.00 -> 64.0 mm
- net Net-(DRGB7-Pad2): track 0.00 -> 62.8 mm
- net Net-(DRGB1-Pad2): track 0.00 -> 58.2 mm, vias 0 -> 2
- net Net-(DRGB2-Pad2): track 0.00 -> 58.1 mm
- net Net-(DRGB3-Pad2): track 0.00 -> 55.1 mm
- net Net-(DRGB10-Pad4): track 0.00 -> 49.5 mm
- net Net-(DRGB4-Pad2): track 0.00 -> 49.0 mm
- net Col11: track 260.7 -> 305.0 mm, vias 2 -> 6
- net Row5: track 385.9 -> 426.2 mm
- net Row1: track 389.0 -> 402.3 mm, vias 0 -> 4
- net Col4: track 150.7 -> 139.0 mm, vias 2 -> 6
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
Commit message: extras wired up, fills started around mcu
Parts:
- CR1, CR2, DR1, QRST1, RGND1, RR1: moved to B.Cu
- moved RGND1 296.0 mm to (89.6, 237.8)
- moved DR1 243.0 mm to (181.5, 298.5)
- moved RR1 219.7 mm to (193.3, 298.3), turned to 270 degrees
- moved CR2 183.9 mm to (186.7, 303.2), turned to 270 degrees
- moved QRST1 179.9 mm to (189.6, 303.3), turned to 270 degrees
- moved CR1 178.6 mm to (191.0, 297.9), turned to 270 degrees
- moved D15 7.42 mm to (70.7, 224.1)
- moved CB5 1.33 mm to (83.6, 229.5)
Connections:
- U2 pad 2: Extra1 -> Extra13
- U2 pad 22: Extra13 -> Extra12
- U2 pad 26: Extra7 -> Extra11
- U2 pad 27: Extra8 -> Extra10
- U2 pad 30: Extra10 -> Extra8
- U2 pad 31: Extra11 -> Extra7
- U2 pad 38: Extra12 -> Extra6
- U2 pad 39: Extra2 -> Extra5
- U2 pad 40: Extra3 -> Extra4
- U2 pad 41: Extra4 -> Extra3
- U2 pad 42: Extra5 -> Extra2
- U2 pad 43: Row1 -> Extra1
- U2 pad 45: Row2 -> Row1
- U2 pad 46: Extra6 -> Row2
Routing:
- net Extra1: track 0.00 -> 37.0 mm
- net Extra2: track 0.00 -> 34.6 mm
- net Extra12: track 0.00 -> 34.1 mm, vias 0 -> 2
- net Extra3: track 0.00 -> 32.1 mm
- net Extra4: track 0.00 -> 30.4 mm
- net Extra5: track 0.00 -> 28.8 mm
- net Extra11: track 0.00 -> 27.6 mm
- net Extra6: track 0.00 -> 27.3 mm
- net Extra10: track 0.00 -> 25.8 mm
- net Extra9: track 0.00 -> 25.1 mm
- net Extra8: track 0.00 -> 24.3 mm
- net Extra7: track 0.00 -> 23.8 mm
- net GNDD: track 0.00 -> 11.6 mm
- net Net-(D15-Pad2): track 11.4 -> 3.44 mm
- net Row2: track 267.2 -> 260.9 mm
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- added copper zone on F.Cu, net 3.3V
- added copper zone on B.Cu, net GNDD

Commit message: Placed... everything? wired everything?
Parts:
- added J2: Conn_ARM_JTAG_SWD_10, sixtyfive:Conn_ARM_JTAG_SWD_10, B.Cu at (53.1, 258.5)
- added SW1: SW_Push, sixtyfive:smdPushBtn, B.Cu at (120.7, 279.6)
- moved QRST1 68.3 mm to (123.5, 285.9)
- moved CR2 68.3 mm to (120.7, 285.8)
- moved CR1 66.0 mm to (127.1, 281.5)
- moved RR1 66.0 mm to (129.4, 281.9)
- moved DR1 60.2 mm to (124.9, 278.0), turned to 90 degrees
Routing:
- net NRST: track 0.00 -> 155.1 mm, vias 0 -> 5
- net 3.3V: track 42.7 -> 163.4 mm, vias 5 -> 6
- net BOOT0: track 0.00 -> 82.3 mm, vias 0 -> 4
- net SWDIO: track 0.00 -> 47.0 mm, vias 0 -> 1
- net SWCLK: track 0.00 -> 46.6 mm, vias 0 -> 2
- net Net-(DR1-Pad2): track 0.00 -> 11.4 mm

Commit message: Switched some components to "basic" parts, hopefully we good
Parts:
- CR1, CR2, CSI1, CSO1: footprint Capacitor_SMD:C_0805_2012Metric_Pad1.15x1.40mm_HandSolder -> Capacitor_SMD:C_0805_2012Metric
- D1, D10, D11, D12, D13, D14, D15, D16, D17, D18, D19, D2, D20, D21, D22, D23, D24, D25, D26, D27, D28, D29, D3, D30, D31, D32, D33, D34, D35, D36, D37, D38, D39, D4, D40, D41, D42, D43, D44, D45, D46, D47, D48, D49, D5, D50, D51, D52, D53, D54, D55, D56, D57, D58, D59, D6, D60, D61, D62, D63, D64, D65, D66, D67, D68, D7, D8, D9: value D_Small -> 1N4148
- MX60: footprint MX_Only:MXOnly-6.25U-Hotswap -> MX_Only:MXOnly-6.25U-Hotswap-ReversedStabilizers
- MX67: footprint MX_Only:MXOnly-2.75U-Hotswap-ReversedStabilizers -> MX_Only:MXOnly-2.75U-Hotswap
- MX68: footprint MX_Only:MXOnly-2.25U-Hotswap-ReversedStabilizers -> MX_Only:MXOnly-2.25U-Hotswap
- RCC1, RCC2, RRGB1, RRGB10, RRGB2, RRGB3, RRGB4, RRGB5, RRGB6, RRGB7, RRGB8, RRGB9, RSH1, RSH2: footprint Resistor_SMD:R_1206_3216Metric -> Resistor_SMD:R_0805_2012Metric
- moved CRGB9 238.9 mm to (372.7, 313.3)
- moved DRGB9 238.9 mm to (368.0, 313.9)
- moved RRGB9 238.9 mm to (375.0, 313.9)
- moved CRGB5 221.4 mm to (532.6, 257.0)
- moved CRGB6 221.4 mm to (534.1, 314.3)
- moved D27 221.4 mm to (519.5, 273.9)
- moved D28 221.4 mm to (543.3, 273.9)
- moved D42 221.4 mm to (567.1, 273.9)
- moved D65 221.4 mm to (567.1, 331.1)
- moved MX64 221.4 mm to (543.3, 327.1)
- moved CB1 221.4 mm to (302.8, 275.0)
- moved CB6 221.4 mm to (292.2, 282.4)
- moved CB7 221.4 mm to (292.2, 283.4)
- moved CSH2 221.4 mm to (282.5, 240.8)
- moved D20 221.4 mm to (386.1, 273.9)
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Routing:
- net Net-(DRGB10-Pad4): track 49.5 -> 67.9 mm
- net Net-(DRGB8-Pad2): track 64.0 -> 48.0 mm
- net 5V: track 606.0 -> 618.1 mm
- net GNDD: track 11.6 -> 22.2 mm
- net Row4: track 319.8 -> 322.0 mm
- net Row5: track 426.2 -> 427.0 mm
- net GND: vias 0 -> 19
- added copper zone on B.Cu, net GND
- added copper zone on F.Cu, net GND
Other:
- board outline added: 305 x 98.6 mm

Commit message: Redoing literally all the routing, switched diodes to common anode
Parts:
- removed D35, D36, D37, D38, D39, D40, D41, D42, D43, D44, D45, D46, D47, D48, D49, D50, D51, D52, D53, D54, D55, D56, D57, D58, D59, D60, D61, D62, D63, D64, D65, D66, D67, D68: 1N4148, Diode_SMD:D_SOD-123
- D1, D10, D11, D12, D13, D14, D15, D16, D17, D18, D19, D2, D20, D21, D22, D23, D24, D25, D26, D27, D28, D29, D3, D30, D31, D32, D33, D34, D4, D5, D6, D7, D8, D9: value 1N4148 -> BAV70; footprint Diode_SMD:D_SOD-123 -> Package_TO_SOT_SMD:SOT-23
- moved D34 181.2 mm to (567.4, 333.6), turned to 270 degrees
- moved D33 167.0 mm to (533.8, 333.6), turned to 270 degrees
- moved D21 138.4 mm to (542.5, 290.7), turned to 270 degrees
- moved D32 134.8 mm to (481.3, 333.6), turned to 270 degrees
- moved D8 125.4 mm to (290.1, 268.6), turned to 270 degrees
- moved D22 123.3 mm to (305.6, 307.3), turned to 270 degrees
- moved D7 118.5 mm to (514.1, 252.7), turned to 270 degrees
- moved D20 105.6 mm to (490.3, 290.7), turned to 270 degrees
- moved D23 102.3 mm to (347.5, 309.8), turned to 270 degrees
- moved D9 102.0 mm to (333.1, 271.8), turned to 270 degrees
- moved D6 99.4 mm to (476.0, 252.7), turned to 270 degrees
- moved D31 93.1 mm to (417.4, 333.6), turned to 270 degrees
- moved D19 86.8 mm to (452.2, 290.7), turned to 270 degrees
- moved D24 84.7 mm to (385.6, 309.8), turned to 270 degrees
- moved D10 83.3 mm to (371.2, 271.8), turned to 270 degrees
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Connections:
- D1 pad 1: Row1 -> Net-(D1-Pad1)
- D10 pad 1: Row1 -> Net-(D10-Pad1)
- D11 pad 1: Row1 -> Net-(D11-Pad1)
- D12 pad 1: Row1 -> Net-(D12-Pad1)
- D13 pad 1: Row1 -> Net-(D13-Pad1)
- D14 pad 1: Row1 -> Net-(D14-Pad1)
- D15 pad 1: Row2 -> Net-(D15-Pad1)
- D16 pad 1: Row2 -> Net-(D16-Pad1)
- D17 pad 1: Row2 -> Net-(D17-Pad1)
- D18 pad 1: Row2 -> Net-(D18-Pad1)
- D19 pad 1: Row2 -> Net-(D19-Pad1)
- D2 pad 1: Row1 -> Net-(D2-Pad1)
- D20 pad 1: Row2 -> Net-(D20-Pad1)
- D21 pad 1: Row2 -> Net-(D21-Pad1)
- D22 pad 1: Row2 -> Net-(D22-Pad1)
- D23 pad 1: Row2 -> Net-(D23-Pad1)
- D24 pad 1: Row2 -> Net-(D24-Pad1)
- D25 pad 1: Row2 -> Net-(D25-Pad1)
- D26 pad 1: Row2 -> Net-(D26-Pad1)
- D27 pad 1: Row2 -> Net-(D27-Pad1)
- D28 pad 1: Row2 -> Net-(D28-Pad1)
- D29 pad 1: Row3 -> Net-(D29-Pad1)
- D3 pad 1: Row1 -> Net-(D3-Pad1)
- D30 pad 1: Row3 -> Net-(D30-Pad1)
- D31 pad 1: Row3 -> Net-(D31-Pad1)
- D32 pad 1: Row3 -> Net-(D32-Pad1)
- D33 pad 1: Row3 -> Net-(D33-Pad1)
- D34 pad 1: Row3 -> Net-(D34-Pad1)
- D4 pad 1: Row1 -> Net-(D4-Pad1)
- D5 pad 1: Row1 -> Net-(D5-Pad1)
- D6 pad 1: Row1 -> Net-(D6-Pad1)
- D7 pad 1: Row1 -> Net-(D7-Pad1)
- D8 pad 1: Row1 -> Net-(D8-Pad1)
- D9 pad 1: Row1 -> Net-(D9-Pad1)
- MX1 pad 2: Net-(D1-Pad2) -> Net-(D1-Pad1)
- MX10 pad 2: Net-(D10-Pad2) -> Net-(D5-Pad2)
- MX11 pad 2: Net-(D11-Pad2) -> Net-(D6-Pad1)
- MX12 pad 2: Net-(D12-Pad2) -> Net-(D6-Pad2)
- MX13 pad 2: Net-(D13-Pad2) -> Net-(D7-Pad1)
- MX14 pad 2: Net-(D14-Pad2) -> Net-(D7-Pad2)
- MX15 pad 2: Net-(D15-Pad2) -> Net-(D8-Pad1)
- MX16 pad 2: Net-(D16-Pad2) -> Net-(D8-Pad2)
- MX17 pad 2: Net-(D17-Pad2) -> Net-(D9-Pad1)
- MX18 pad 2: Net-(D18-Pad2) -> Net-(D9-Pad2)
- MX19 pad 2: Net-(D19-Pad2) -> Net-(D10-Pad1)
- MX2 pad 2: Net-(D2-Pad2) -> Net-(D1-Pad2)
- MX20 pad 2: Net-(D20-Pad2) -> Net-(D10-Pad2)
- MX21 pad 2: Net-(D21-Pad2) -> Net-(D11-Pad1)
- MX22 pad 2: Net-(D22-Pad2) -> Net-(D11-Pad2)
- MX23 pad 2: Net-(D23-Pad2) -> Net-(D12-Pad1)
- MX24 pad 2: Net-(D24-Pad2) -> Net-(D12-Pad2)
- MX25 pad 2: Net-(D25-Pad2) -> Net-(D13-Pad1)
- MX26 pad 2: Net-(D26-Pad2) -> Net-(D13-Pad2)
- MX27 pad 2: Net-(D27-Pad2) -> Net-(D14-Pad1)
- MX28 pad 2: Net-(D28-Pad2) -> Net-(D14-Pad2)
- MX29 pad 2: Net-(D29-Pad2) -> Net-(D15-Pad1)
- MX3 pad 2: Net-(D3-Pad2) -> Net-(D2-Pad1)
- MX30 pad 2: Net-(D30-Pad2) -> Net-(D15-Pad2)
- MX31 pad 2: Net-(D31-Pad2) -> Net-(D16-Pad1)
- MX32 pad 2: Net-(D32-Pad2) -> Net-(D16-Pad2)
- MX33 pad 2: Net-(D33-Pad2) -> Net-(D17-Pad1)
- MX34 pad 2: Net-(D34-Pad2) -> Net-(D17-Pad2)
- MX35 pad 2: Net-(D35-Pad2) -> Net-(D18-Pad1)
- MX36 pad 2: Net-(D36-Pad2) -> Net-(D18-Pad2)
- MX37 pad 2: Net-(D37-Pad2) -> Net-(D19-Pad1)
- MX38 pad 2: Net-(D38-Pad2) -> Net-(D19-Pad2)
- MX39 pad 2: Net-(D39-Pad2) -> Net-(D20-Pad1)
- MX4 pad 2: Net-(D4-Pad2) -> Net-(D2-Pad2)
- MX40 pad 2: Net-(D40-Pad2) -> Net-(D20-Pad2)
- MX41 pad 2: Net-(D41-Pad2) -> Net-(D21-Pad1)
- MX42 pad 2: Net-(D42-Pad2) -> Net-(D21-Pad2)
- MX43 pad 2: Net-(D43-Pad2) -> Net-(D22-Pad1)
- MX44 pad 2: Net-(D44-Pad2) -> Net-(D22-Pad2)
- MX45 pad 2: Net-(D45-Pad2) -> Net-(D23-Pad1)
- MX46 pad 2: Net-(D46-Pad2) -> Net-(D23-Pad2)
- MX47 pad 2: Net-(D47-Pad2) -> Net-(D24-Pad1)
- MX48 pad 2: Net-(D48-Pad2) -> Net-(D24-Pad2)
- MX49 pad 2: Net-(D49-Pad2) -> Net-(D25-Pad1)
- MX5 pad 2: Net-(D5-Pad2) -> Net-(D3-Pad1)
- MX50 pad 2: Net-(D50-Pad2) -> Net-(D25-Pad2)
- MX51 pad 2: Net-(D51-Pad2) -> Net-(D26-Pad1)
- MX52 pad 2: Net-(D52-Pad2) -> Net-(D26-Pad2)
- MX53 pad 2: Net-(D53-Pad2) -> Net-(D27-Pad1)
- MX54 pad 2: Net-(D54-Pad2) -> Net-(D27-Pad2)
- MX55 pad 2: Net-(D55-Pad2) -> Net-(D28-Pad1)
- MX56 pad 2: Net-(D56-Pad2) -> Net-(D28-Pad2)
- MX57 pad 2: Net-(D57-Pad2) -> Net-(D29-Pad1)
- MX58 pad 2: Net-(D58-Pad2) -> Net-(D29-Pad2)
- MX59 pad 2: Net-(D59-Pad2) -> Net-(D30-Pad1)
- MX6 pad 2: Net-(D6-Pad2) -> Net-(D3-Pad2)
- MX60 pad 2: Net-(D60-Pad2) -> Net-(D31-Pad1)
- MX61 pad 2: Net-(D61-Pad2) -> Net-(D32-Pad1)
- MX62 pad 2: Net-(D62-Pad2) -> Net-(D32-Pad2)
- MX63 pad 2: Net-(D63-Pad2) -> Net-(D33-Pad1)
- MX64 pad 2: Net-(D64-Pad2) -> Net-(D33-Pad2)
- MX65 pad 2: Net-(D65-Pad2) -> Net-(D34-Pad1)
- MX66 pad 2: Net-(D66-Pad2) -> Net-(D34-Pad2)
- MX67 pad 2: Net-(D67-Pad2) -> Net-(D30-Pad2)
- MX68 pad 2: Net-(D68-Pad2) -> Net-(D31-Pad2)
- MX69 pad 2: Net-(D60-Pad2) -> Net-(D31-Pad1)
- MX7 pad 2: Net-(D7-Pad2) -> Net-(D4-Pad1)
- MX8 pad 2: Net-(D8-Pad2) -> Net-(D4-Pad2)
- MX9 pad 2: Net-(D9-Pad2) -> Net-(D5-Pad1)
Routing:
- net Row4: track 322.0 -> 0.00 mm, vias 16 -> 0
- net Col14: track 362.0 -> 87.6 mm, vias 6 -> 5
- net Col13: track 346.8 -> 114.1 mm, vias 6 -> 5
- net Row1: track 404.0 -> 190.5 mm, vias 4 -> 0
- net Col12: track 325.2 -> 116.6 mm, vias 6 -> 5
- net Col11: track 305.0 -> 118.9 mm, vias 6 -> 5
- net Col10: track 274.0 -> 109.5 mm, vias 6 -> 5
- net NRST: track 155.1 -> 2.89 mm, vias 5 -> 0
- net Col9: track 252.0 -> 102.3 mm, vias 6 -> 5
- net Row3: track 301.1 -> 152.4 mm, vias 26 -> 0
- net 3.3V: track 163.4 -> 19.4 mm, vias 6 -> 0
- net Row5: track 427.0 -> 286.0 mm
- net Col2: track 107.8 -> 0.00 mm
- net Net-(DRGB5-Pad2): track 103.9 -> 0.00 mm, vias 2 -> 0
- net BOOT0: track 82.3 -> 4.59 mm, vias 4 -> 0
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
Commit message: Rerouted everything, feels cleaner now?
Parts:
- DS1: value RB060M-60TR -> SM4007; footprint Diode_SMD:D_SOD-123 -> Diode_SMD:D_SOD-123F
- RSI1: value 100k -> 1M; footprint Resistor_SMD:R_1206_3216Metric -> Resistor_SMD:R_0805_2012Metric
- moved J2 76.3 mm to (341.8, 328.4)
- moved SW1 48.5 mm to (386.2, 326.5), turned to 90 degrees
- moved CR2 44.8 mm to (382.5, 332.5)
- moved QRST1 44.8 mm to (385.3, 332.5)
- moved D1 44.2 mm to (304.4, 250.2), turned to 0 degrees
- moved DR1 40.3 mm to (382.1, 325.1), turned to 90 degrees
- moved CR1 35.7 mm to (379.9, 325.9), turned to 90 degrees
- moved RR1 31.2 mm to (377.6, 325.4), turned to 90 degrees
- moved RS1 18.8 mm to (315.4, 271.3), turned to 270 degrees
- moved RS2 18.6 mm to (313.1, 271.3)
- moved RSI1 17.1 mm to (287.8, 255.5), turned to 180 degrees
- moved D30 12.6 mm to (336.7, 321.6)
- moved F1 9.53 mm to (276.2, 257.3)
- moved DF1 9.50 mm to (279.5, 257.9)
- moved CSI1 9.40 mm to (281.7, 258.6)
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Connections:
- U2 pad 19: Row5 -> Row4
- U2 pad 20: Row4 -> Row5
Routing:
- net Row4: track 0.00 -> 279.7 mm, vias 0 -> 2
- net Col14: track 87.6 -> 351.8 mm, vias 5 -> 6
- net Col13: track 114.1 -> 347.8 mm, vias 5 -> 6
- net BOOT0: track 4.59 -> 223.2 mm, vias 0 -> 2
- net 3.3V: track 19.4 -> 232.9 mm, vias 0 -> 7
- net NRST: track 2.89 -> 215.8 mm, vias 0 -> 2
- net Col12: track 116.6 -> 320.2 mm, vias 5 -> 6
- net Col11: track 118.9 -> 304.5 mm, vias 5 -> 6
- net Col10: track 109.5 -> 276.8 mm, vias 5 -> 6
- net SWCLK: track 0.00 -> 159.3 mm, vias 0 -> 2
- net SWDIO: track 0.00 -> 156.4 mm, vias 0 -> 2
- net Col9: track 102.3 -> 251.9 mm, vias 5 -> 6
- net Col2: track 0.00 -> 123.0 mm, vias 5 -> 6
- net Row3: track 152.4 -> 258.8 mm, vias 0 -> 2
- net Net-(DRGB5-Pad2): track 0.00 -> 100.0 mm, vias 0 -> 2
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Other:
- board size 305 x 98.6 mm -> 305 x 100.3 mm
- net class Switch added: clearance 0.2, trace_width 0.25, via_dia 0.5, via_drill 0.3
