File: sixtyfive.sch (KiCad schematic (older format))
At the start: 169 parts, among them J1 Conn_01x12, J2 STLINK_6_Pin, Q1 BSS138, SW1 SW_Push, U1 SRV05-4, U2 STM32F072C8Tx, U3 MCP1700-3302E_SOT23

Commit message: Further clarified schematic
Connections:
- net 3.3V is gone; now on net +3V3: CSO1.1, DS1.2 (A), J2.1 (3.3V), Q1.1 (G), RS2.1, SW1.1, U3.2 (VO)
Other:
- moved on the sheet: CB7
Changed lines of the file:
@@
 Wire Wire Line
 	25050 21800 25050 21650
-Text GLabel 25800 20850 2    50   Output ~ 0
-3.3V
 Text GLabel 23500 20850 0    50   Input ~ 0
 VBUS
@@
 L Device:C_Small CB7
 U 1 1 5F16FFEF
-P 31650 16600
-F 0 "CB7" H 31742 16646 50  0000 L CNN
-F 1 "100n" H 31742 16555 50  0000 L CNN
-F 2 "Capacitor_SMD:C_0402_1005Metric" H 31650 16600 50  0001 C CNN
-F 3 "~" H 31650 16600 50  0001 C CNN
-F 4 "C1525" H 31650 16600 50  0001 C CNN "JLCCode"
-	1    31650 16600
+P 31600 16600
+F 0 "CB7" H 31692 16646 50  0000 L CNN
+F 1 "100n" H 31692 16555 50  0000 L CNN
+F 2 "Capacitor_SMD:C_0402_1005Metric" H 31600 16600 50  0001 C CNN
+F 3 "~" H 31600 16600 50  0001 C CNN
+F 4 "C1525" H 31600 16600 50  0001 C CNN "JLCCode"
+	1    31600 16600
 	1    0    0    -1
 $EndComp
@@
 Text GLabel 30350 10350 1    50   Input ~ 0
 Col14
-Text GLabel 21750 20750 0    50   Input ~ 0
-3.3V
 $Comp
 L power:GND #PWR0114
@@
 F 3 "" H 20900 18350 50  0001 C CNN
 	1    20900 18350
-	0    -1   -1   0
+	1    0    0    -1
 $EndComp
 Wire Wire Line
@@
 	19650 18250 19500 18250
 $Comp
-L power:GND #PWR0118
-U 1 1 602C0E60
-P 19500 18100
-F 0 "#PWR0118" H 19500 17850 50  0001 C CNN
-F 1 "GND" V 19505 17972 50  0000 R CNN
-F 2 "" H 19500 18100 50  0001 C CNN
-F 3 "" H 19500 18100 50  0001 C CNN
-	1    19500 18100
-	0    1    1    0
-$EndComp
-$Comp
 L power:GND #PWR0119
 U 1 1 602C20E9
@@
 F 3 "" H 19500 18250 50  0001 C CNN
 	1    19500 18250
-	0    1    1    0
+	1    0    0    -1
 $EndComp
 $Comp
@@
 Wire Wire Line
 	20300 19450 20300 19500
-Text GLabel 20300 19500 3    50   Input ~ 0
-3.3V
 $Comp
 L LED:WS2812B DRGB5
@@
 Text GLabel 6300 18200 1    50   Input ~ 0
 5V
-Text GLabel 5850 18200 1    50   Input ~ 0
-3.3V
 Text GLabel 5650 19350 0    50   Input ~ 0
 RGB_3V3
@@
 L power:+3.3V #PWR0103
 U 1 1 5FE0A1ED
-P 31000 16450
-F 0 "#PWR0103" H 31000 16300 50  0001 C CNN
-F 1 "+3.3V" H 31015 16623 50  0000 C CNN
-F 2 "" H 31000 16450 50  0001 C CNN
-F 3 "" H 31000 16450 50  0001 C CNN
-	1    31000 16450
-	1    0    0    -1
-$EndComp
-$Comp
-L power:+3.3V #PWR0110
-U 1 1 5FEFAC78
-P 31650 16450
-F 0 "#PWR0110" H 31650 16300 50  0001 C CNN
-F 1 "+3.3V" H 31665 16623 50  0000 C CNN
-F 2 "" H 31650 16450 50  0001 C CNN
-F 3 "" H 31650 16450 50  0001 C CNN
-	1    31650 16450
+P 31200 16400
+F 0 "#PWR0103" H 31200 16250 50  0001 C CNN
+F 1 "+3.3V" H 31215 16573 50  0000 C CNN
+F 2 "" H 31200 16400 50  0001 C CNN
+F 3 "" H 31200 16400 50  0001 C CNN
+	1    31200 16400
 	1    0    0    -1
 $EndComp
@@
 L power:GNDD #PWR0111
 U 1 1 60506036
-P 31000 16750
-F 0 "#PWR0111" H 31000 16500 50  0001 C CNN
-F 1 "GNDD" H 31004 16595 50  0000 C CNN
-F 2 "" H 31000 16750 50  0001 C CNN
-F 3 "" H 31000 16750 50  0001 C CNN
-	1    31000 16750
-	1    0    0    -1
-$EndComp
-$Comp
-L power:GNDD #PWR0145
-U 1 1 60506325
-P 31650 16750
-F 0 "#PWR0145" H 31650 16500 50  0001 C CNN
-F 1 "GNDD" H 31654 16595 50  0000 C CNN
-F 2 "" H 31650 16750 50  0001 C CNN
-F 3 "" H 31650 16750 50  0001 C CNN
-	1    31650 16750
+P 31200 16800
+F 0 "#PWR0111" H 31200 16550 50  0001 C CNN
+F 1 "GNDD" H 31204 16645 50  0000 C CNN
+F 2 "" H 31200 16800 50  0001 C CNN
+F 3 "" H 31200 16800 50  0001 C CNN
+	1    31200 16800
 	1    0    0    -1
 $EndComp
@@
 Wire Wire Line
 	29000 15750 29100 15750
-Text HLabel 30350 16500 0    50   Input ~ 0
-VBAT
-Text HLabel 30350 16700 0    50   Input ~ 0
-VSS
 Wire Wire Line
 	30800 16500 30800 16450
 Wire Wire Line
-	30800 16450 31000 16450
-Wire Wire Line
 	31200 16450 31200 16500
 Wire Wire Line
@@
 Wire Wire Line
 	30800 16750 30800 16700
-Connection ~ 31000 16750
-Wire Wire Line
-	31000 16750 30800 16750
-Wire Wire Line
-	31000 16750 31200 16750
-Connection ~ 31000 16450
-Wire Wire Line
-	31000 16450 31200 16450
-Wire Wire Line
-	31650 16450 31650 16500
-Wire Wire Line
-	31650 16700 31650 16750
 Wire Wire Line
 	30350 16700 30350 16750
@@
 Wire Wire Line
 	31150 17350 30950 17350
+Text Label 31100 17350 2    50   ~ 0
+VDDIO2
+Text Label 31200 16450 2    50   ~ 0
+VDD
+Text Label 30300 17350 2    50   ~ 0
+VDDA
+Wire Wire Line
+	31200 16750 31600 16750
+Wire Wire Line
+	31600 16750 31600 16700
+Connection ~ 31200 16750
+Wire Wire Line
+	31200 16450 31600 16450
+Wire Wire Line
+	31600 16450 31600 16500
+Connection ~ 31200 16450
+Wire Wire Line
+	30800 16750 31200 16750
+Wire Wire Line
+	30800 16450 31200 16450
+Wire Wire Line
+	31200 16450 31200 16400
+Wire Wire Line
+	31200 16750 31200 16800
+Text Label 30350 16500 2    50   ~ 0
+VBAT
+$Comp
+L power:+3.3V #PWR0110
+U 1 1 60B95B95
+P 21700 20750
+F 0 "#PWR0110" H 21700 20600 50  0001 C CNN
+F 1 "+3.3V" V 21715 20878 50  0000 L CNN
+F 2 "" H 21700 20750 50  0001 C CNN
+F 3 "" H 21700 20750 50  0001 C CNN
+	1    21700 20750
+	0    -1   -1   0
+$EndComp
+Wire Wire Line
+	21700 20750 21750 20750
+Wire Wire Line
+	19500 18250 19500 18100
+Connection ~ 19500 18250
+$Comp
+L power:+3.3V #PWR0118
+U 1 1 60D3228E
+P 20050 19450
+F 0 "#PWR0118" H 20050 19300 50  0001 C CNN
+F 1 "+3.3V" H 20065 19623 50  0000 C CNN
+F 2 "" H 20050 19450 50  0001 C CNN
+F 3 "" H 20050 19450 50  0001 C CNN
+	1    20050 19450
+	1    0    0    -1
+$EndComp
+Wire Wire Line
+	20050 19500 20050 19450
+Wire Wire Line
+	20050 19500 20300 19500
+$Comp
+L power:+3.3V #PWR0145
+U 1 1 60D9DF7D
+P 5850 18200
+F 0 "#PWR0145" H 5850 18050 50  0001 C CNN
+F 1 "+3.3V" H 5865 18373 50  0000 C CNN
+F 2 "" H 5850 18200 50  0001 C CNN
+F 3 "" H 5850 18200 50  0001 C CNN
+	1    5850 18200
+	1    0    0    -1
+$EndComp
+$Comp
+L power:+3.3V #PWR?
+U 1 1 60DA260B
+P 25800 20750
+F 0 "#PWR?" H 25800 20600 50  0001 C CNN
+F 1 "+3.3V" H 25815 20923 50  0000 C CNN
+F 2 "" H 25800 20750 50  0001 C CNN
+F 3 "" H 25800 20750 50  0001 C CNN
+	1    25800 20750
+	1    0    0    -1
+$EndComp
+Wire Wire Line
+	25800 20750 25800 20850
 $EndSCHEMATC
